Commit message: walk on plane

File: src/holosoma_retargeting/demo_data/climb/mocap_climb_seq_0/multi_boxes.urdf (robot description, URDF)
Before this commit: robot multi_boxes, 4 links, 3 joints
Links:
- added link planes_link, mass 33.33; collision mesh filename=box_models/meshes_all.obj scale=0.7415730337078652 0.7415730337078652 0.7415730337078652; visual mesh filename=box_models/meshes_all.obj scale=0.7415730337078652 0.7415730337078652 0.7415730337078652
Joints:
- added joint world_to_planes: type fixed, parent world, child planes_link, origin xyz=0 0 0 rpy=0 0 0

File: src/holosoma_retargeting/demo_data/scene/sequence_07/scene.urdf (robot description, URDF)
Before this commit: robot scene, 2 links, 1 joints
Links:
- removed link scene_link
- added link multi_boxes_link, mass 33.33; collision mesh filename=box_models/box1.obj scale=0.7415730337078652 0.7415730337078652 0.7415730337078652; visual mesh filename=box_models/box1.obj scale=0.7415730337078652 0.7415730337078652 0.7415730337078652
Joints:
- removed joint world_to_scene
- added joint world_to_multi_boxes: type fixed, parent world, child multi_boxes_link, origin xyz=0 0 0 rpy=0 0 0

Commit message: run stair sequence with all planes

File: src/holosoma_retargeting/demo_data/climb/mocap_climb_seq_0/multi_boxes.urdf (robot description, URDF)
Before this commit: robot multi_boxes, 5 links, 4 joints
Links:
- removed link box2_link
- removed link box3_link
- removed link multi_boxes_link
Joints:
- removed joint world_to_box2
- removed joint world_to_box3
- removed joint world_to_multi_boxes
